Commit message: mapping_navigation

File: asv_wave_sim_gazebo/models/boatcleaningc/urdf/boatcleaningc.urdf (robot description, URDF)
Before this commit: robot boatcleaningc, 7 links, 6 joints
Links:
- link axedroit: geometry collision mesh filename=package://asv_wave_sim_gazebo/models/boatcleaningc/meshes/a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; visual mesh filename=package://asv_wave_sim_gazebo/models/boatcleaningc/meshes/a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
- link axegauche: geometry collision mesh filename=package://asv_wave_sim_gazebo/models/boatcleaningc/meshes/a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; visual mesh filename=package://asv_wave_sim_gazebo/models/boatcleaningc/meshes/a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
- link baseboatclening: geometry collision mesh filename=package://asv_wave_sim_gazebo/models/boatcleaningc/meshes/b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; visual mesh filename=package://asv_wave_sim_gazebo/models/boatcleaningc/meshes/b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
- link fandroit: geometry collision mesh filename=package://asv_wave_sim_gazebo/models/boatcleaningc/meshes/f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; visual mesh filename=package://asv_wave_sim_gazebo/models/boatcleaningc/meshes/f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
- link fangauche: geometry collision mesh filename=package://asv_wave_sim_gazebo/models/boatcleaningc/meshes/f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; visual mesh filename=package://asv_wave_sim_gazebo/models/boatcleaningc/meshes/f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
